File: mainboard/LED-Ring.kicad_sch (KiCad schematic)
At the start: 64 parts

Commit message: Rearranged LEDs
Parts:
- removed C31, C32, C33, C34, C35: 0.1uF, Capacitor_SMD:C_0603_1608Metric, symbol Device:C_Small
- removed D10, D11, D12, D13, D14, D15, D16, D17, D18, D19, D20, D21, D22, D23, D24, D25, D26, D27, D28, D29, D30, D31, D32, D33, D34, D35, D4, D5, D6, D7, D8, D9: WS2812B-2020, LED_SMD:LED_WS2812B-2020_PLCC4_2.0x2.0mm, symbol LED:SK6812MINI
- added LED10, LED11, LED12, LED13, LED14, LED15, LED16, LED17, LED18, LED19, LED20, LED21, LED22, LED23, LED24, LED25, LED26, LED27, LED28, LED29, LED30, LED4, LED5, LED6, LED7, LED8, LED9: WS2812B-2020, PhiMai:LED_WS2812B-2020_PLCC4_2.0x2.0mm, symbol LED:WS2812B-2020
Connections:
- net +5V: now also LED10.4 (VDD), LED11.4 (VDD), LED12.4 (VDD), LED13.4 (VDD), LED14.4 (VDD), LED15.4 (VDD), LED16.4 (VDD), LED17.4 (VDD), LED18.4 (VDD), LED19.4 (VDD), LED20.4 (VDD), LED21.4 (VDD), LED22.4 (VDD), LED23.4 (VDD), LED24.4 (VDD), LED25.4 (VDD), LED26.4 (VDD), LED27.4 (VDD), LED28.4 (VDD), LED29.4 (VDD), LED30.4 (VDD), LED4.4 (VDD), LED5.4 (VDD), LED6.4 (VDD), LED7.4 (VDD), LED8.4 (VDD), LED9.4 (VDD)
- net GND: now also LED10.2 (VSS), LED11.2 (VSS), LED12.2 (VSS), LED13.2 (VSS), LED14.2 (VSS), LED15.2 (VSS), LED16.2 (VSS), LED17.2 (VSS), LED18.2 (VSS), LED19.2 (VSS), LED20.2 (VSS), LED21.2 (VSS), LED22.2 (VSS), LED23.2 (VSS), LED24.2 (VSS), LED25.2 (VSS), LED26.2 (VSS), LED27.2 (VSS), LED28.2 (VSS), LED29.2 (VSS), LED30.2 (VSS), LED4.2 (VSS), LED5.2 (VSS), LED6.2 (VSS), LED7.2 (VSS), LED8.2 (VSS), LED9.2 (VSS)
- net LED_DATA_5V_AFTER_KEYS: now also LED4.3 (DIN)
- new net: LED24.1 (DOUT), LED25.3 (DIN)
- new net: LED23.1 (DOUT), LED24.3 (DIN)
- new net: LED14.1 (DOUT), LED15.3 (DIN)
- new net: LED13.1 (DOUT), LED14.3 (DIN)
- new net: LED15.1 (DOUT), LED16.3 (DIN)
- new net: LED19.1 (DOUT), LED20.3 (DIN)
- new net: LED18.1 (DOUT), LED19.3 (DIN)
- new net: LED6.1 (DOUT), LED7.3 (DIN)
- new net: LED5.1 (DOUT), LED6.3 (DIN)
- new net: LED10.3 (DIN), LED9.1 (DOUT)
- new net: LED8.1 (DOUT), LED9.3 (DIN)
- new net: LED28.1 (DOUT), LED29.3 (DIN)
- new net: LED27.1 (DOUT), LED28.3 (DIN)
- new net: LED7.1 (DOUT), LED8.3 (DIN)
- new net: LED17.1 (DOUT), LED18.3 (DIN)
- new net: LED22.1 (DOUT), LED23.3 (DIN)
- new net: LED21.1 (DOUT), LED22.3 (DIN)
- new net: LED11.1 (DOUT), LED12.3 (DIN)
- new net: LED10.1 (DOUT), LED11.3 (DIN)
- new net: LED29.1 (DOUT), LED30.3 (DIN)
- new net: LED4.1 (DOUT), LED5.3 (DIN)
- new net: LED16.1 (DOUT), LED17.3 (DIN)
- new net: LED20.1 (DOUT), LED21.3 (DIN)
- new net: LED26.1 (DOUT), LED27.3 (DIN)
- new net: LED25.1 (DOUT), LED26.3 (DIN)
- new net: LED12.1 (DOUT), LED13.3 (DIN)
- no-connect marks 1 -> 3
