File: mainboard/VolumepadMainboard.kicad_sch (KiCad schematic)
At the start: 94 parts, among them J1 USB_C_Receptacle_USB2.0, J2 BLDC, J3 USB_Extension_Board, J4 Touch_Extension_Board, Q1 MMBT4403, Q2 2N7002, SW1 SW_Push, SW2 SW_Push, SW3 SW_Push, SW4 SW_Push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

Commit message: Removed the onboard USB-C plug and added a display connector
Parts:
- added J5: Display_Connector, Connector_JST:JST_GH_BM08B-GHS-TBT_1x08-1MP_P1.25mm_Vertical, symbol Connector:Conn_01x08_Pin
- added R27, R28: 33, Resistor_SMD:R_0603_1608Metric, symbol Device:R_Small
- DS1, J1, R1, R2, R23, R24, U6: now not fitted; now left out of the parts list
- JP1, JP2: now not fitted
Connections:
- net +3V3: now also J5.7 (Pin_7)
- net +5V: now also J3.1 (Pin_1), J3.2 (Pin_2); no longer J3.4 (Pin_4), J3.6 (Pin_6)
- net Aux_USB_D+: now also J3.5 (Pin_5), U1.14 (USB_D+); no longer J3.3 (Pin_3)
- net Aux_USB_D-: now also J3.4 (Pin_4), U1.13 (USB_D-); no longer J3.2 (Pin_2)
- net GND: now also J3.3 (Pin_3), J3.6 (Pin_6), J5.8 (Pin_8); no longer J3.1 (Pin_1), J3.5 (Pin_5)
- net LCD_CS: now also J5.2 (Pin_2)
- net LCD_DC: now also J5.3 (Pin_3)
- net LCD_MOSI: now also R27.2
- net LCD_RST: now also J5.4 (Pin_4)
- net LCD_SCK: now also R28.2
- net Protected_USB_D+: no longer U1.14 (USB_D+)
- net Protected_USB_D-: no longer U1.13 (USB_D-)
- net at Q2.3 (D): now also J5.1 (Pin_1); no longer DS1.8 (BL)
- new net: J5.5 (Pin_5), R27.1
- new net: J5.6 (Pin_6), R28.1
Other:
- moved on the sheet: J4, Q2, R21, R22, R25, R26

Commit message: Rearranged LEDs
Parts:
- removed D1, D2, D3: SK6812MINI-E, LED_SMD:LED_SK6812MINI_PLCC4_3.5x3.5mm_P1.75mm, symbol LED:SK6812MINI
- removed DS1: TFT_2.25_ST7789, PhiMai:TFT_2.25_ST7789_1x08_2.54mm, symbol PhiMai:TFT_2.25_ST7789
- removed R23, R24: 33, Resistor_SMD:R_0603_1608Metric, symbol Device:R_Small
- added D1: ORANGE, LED_SMD:LED_0805_2012Metric, symbol Device:LED
- added D2: GREEN, LED_SMD:LED_0805_2012Metric, symbol Device:LED
- added D3: BLUE, LED_SMD:LED_0805_2012Metric, symbol Device:LED
- added JP3, JP4, JP5: Standby Jumper, Jumper:SolderJumper-2_P1.3mm_Bridged_RoundedPad1.0x1.5mm, symbol Jumper:Jumper_2_Bridged
- added LED1, LED2, LED3: MX_SK6812MINI-E, PCM_marbastlib-mx:LED_MX_6028R, symbol PCM_marbastlib-mx:MX_SK6812MINI-E
- added R29: 330, Resistor_SMD:R_0603_1608Metric, symbol Device:R_Small
- added R30: 2.2k, Resistor_SMD:R_0603_1608Metric, symbol Device:R_Small
- added R31: 1k, Resistor_SMD:R_0603_1608Metric, symbol Device:R_Small
- C51: footprint Capacitor_SMD:C_1206_3216Metric -> Capacitor_SMD:C_0805_2012Metric
- H2: footprint MountingHole:MountingHole_2.7mm_M2.5_Pad_Via -> MountingHole:MountingHole_3.2mm_M3_Pad_Via
- L1: footprint Inductor_SMD:L_0603_1608Metric -> Inductor_SMD:L_0805_2012Metric
Connections:
- net +3V3: now also JP5.2 (B)
- net +5V: now also JP4.2 (B), LED1.1 (VDD), LED2.1 (VDD), LED3.1 (VDD)
- net Aux_USB_D+: now also J3.4 (Pin_4); no longer J3.5 (Pin_5)
- net Aux_USB_D-: now also J3.5 (Pin_5); no longer J3.4 (Pin_4)
- net GND: now also LED1.4 (VSS), LED2.4 (VSS), LED3.4 (VSS), R29.2, R30.2, R31.2
- net LED_DATA_5V_AFTER_KEYS: now also LED3.2 (DOUT)
- net MOTOR_DIAG: now also JP3.2 (B)
- net at R12.2: now also LED1.3 (DIN)
- new net: D3.1 (K), R31.1
- new net: D3.2 (A), JP5.1 (A)
- new net: D2.2 (A), JP4.1 (A)
- new net: D2.1 (K), R30.1
- new net: LED1.2 (DOUT), LED2.3 (DIN)
- new net: D1.1 (K), R29.1
- new net: D1.2 (A), JP3.1 (A)
- new net: LED2.2 (DOUT), LED3.3 (DIN)
