File: lcd-display.kicad_sch (KiCad schematic)
At the start: 11 parts, among them J901 Conn_01x08_Socket, Q901 AO3400A

Commit message: Started adding LCSC part numbers to make ordering the parts easier
Parts:
- J901: now left out of the parts list
Changed lines of the file:
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@@
 		(body_style 1)
 		(exclude_from_sim no)
-		(in_bom yes)
+		(in_bom no)
 		(on_board yes)
 		(in_pos_files yes)
