File: leds.kicad_sch (KiCad schematic)
At the start: 4 parts, among them U601 74AHCT1G125

Commit message: Started adding LCSC part numbers to make ordering the parts easier
Parts:
- C601: LCSC (none) -> C42405541
Changed lines of the file:
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@@
+			)
+		)
+		(property "LCSC" "C42405541"
+			(at 59.69 46.99 0)
+			(hide yes)
+			(show_name no)
+			(do_not_autoplace no)
+			(effects
+				(font
+					(size 1.27 1.27)
+				)
 			)
 		)
